Commit message: navigation by diff drive

File: urdf/robot.urdf (robot description, URDF)
Before this commit: robot frame_robot, 1 links, 14 joints
Links:
- added link base_link; visual box size=0 0 0
Joints:
- added joint Base_to_base: type fixed, parent base_footprint, child base_link
- joint front_links_joint: parent base_footprint -> base_link
- joint left_links_joint: origin (none) -> xyz=0 0 0 rpy=0 0 0; parent base_footprint -> base_link
- joint lidar_joint: parent base_footprint -> base_link
- joint middle_links_joint: parent base_footprint -> base_link
- joint rear_links_joint: parent base_footprint -> base_link
- joint right_links_joint: parent base_footprint -> base_link
- joint wheel_support_1_joint: parent base_footprint -> base_link
- joint wheel_support_2_joint: parent base_footprint -> base_link
- joint wheel_support_3_joint: parent base_footprint -> base_link
- joint wheel_support_4_joint: parent base_footprint -> base_link
- joint wheels_bl_joint: origin xyz=-0.175 -0.175 0 rpy=0 0 0 -> xyz=-0.175 0.175 0 rpy=0 0 0; parent base_footprint -> base_link
- joint wheels_br_joint: origin xyz=0.175 -0.175 0 rpy=0 0 0 -> xyz=-0.175 -0.175 0 rpy=0 0 0; parent base_footprint -> base_link
- joint wheels_fl_joint: origin xyz=-0.175 0.175 0 rpy=0 0 0 -> xyz=0.175 0.175 0 rpy=0 0 0; parent base_footprint -> base_link
- joint wheels_fr_joint: origin xyz=0.175 0.175 0 rpy=0 0 0 -> xyz=0.175 -0.175 0 rpy=0 0 0; parent base_footprint -> base_link
