Commit message: differential drive done

File: urdf/robot_omni.urdf (robot description, URDF)
Before this commit: robot frame_robot, 2 links, 15 joints
Links:
- link base_link: geometry visual box size=0.001 0.001 0.001
Joints:
- removed joint front_links_joint
- removed joint left_links_joint
- removed joint lidar_joint
- removed joint middle_links_joint
- removed joint rear_links_joint
- removed joint right_links_joint
- removed joint wheel_support_1_joint
- removed joint wheel_support_2_joint
- removed joint wheel_support_3_joint
- removed joint wheel_support_4_joint
- removed joint wheels_bl_joint
- removed joint wheels_br_joint
- removed joint wheels_fl_joint
- removed joint wheels_fr_joint
